File: SL_Christmas_Tree_B/SL_Christmas_Tree_B.kicad_pcb (KiCad board)
At the start: 2 copper layers, 85.7 x 116 mm, 64 parts

Commit message: v2.1 Final
Parts:
- moved C203 53.4 mm to (109.7, 118.7)
- moved C213 50.2 mm to (92.3, 141.5), turned to 0 degrees
- moved C202 47.2 mm to (115.4, 136.6)
- moved C204 44.1 mm to (107.9, 104.7)
- moved C212 42.6 mm to (87.5, 136.2), turned to 0 degrees
- moved C209 41.9 mm to (92.7, 105.8), turned to 0 degrees
- moved C205 39.1 mm to (106.3, 92.8)
- moved C210 38.9 mm to (91.8, 114.4), turned to 0 degrees
- moved C211 37.3 mm to (87.1, 123.3), turned to 0 degrees
- moved C206 34.8 mm to (106.5, 79.4)
- moved C201 32.8 mm to (113.8, 147.9)
- moved C208 32.5 mm to (95.8, 80.8), turned to 0 degrees
- moved C105 11.0 mm to (105.5, 142.4), turned to 180 degrees
- moved C106 8.97 mm to (106.0, 154.6), turned to 180 degrees
- moved C109 5.05 mm to (92.6, 129.7)
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Routing:
- net GND: track 0.28 -> 1115.2 mm, vias 58 -> 89
- net +5V: track 263.9 -> 583.3 mm, vias 8 -> 9
- net Net-(D208-DIN): track 0.00 -> 30.3 mm
- net Net-(D102-DOUT): track 0.00 -> 25.5 mm
- net Net-(D204-DOUT): track 0.00 -> 24.8 mm
- net Net-(D205-DOUT): track 0.00 -> 21.4 mm
- net Net-(D113-DOUT): track 0.00 -> 19.6 mm
- net Net-(D210-DOUT): track 0.00 -> 19.0 mm
- net Net-(D112-DOUT): track 0.00 -> 18.6 mm
- net Net-(D201-DOUT): track 0.00 -> 18.5 mm
- net Net-(D101-DIN): track 0.00 -> 18.1 mm
- net Net-(D212-DOUT): track 0.00 -> 17.6 mm
- net Net-(D108-DOUT): track 0.00 -> 15.5 mm
- net Net-(D109-DOUT): track 0.00 -> 14.2 mm
- net Net-(D203-DOUT): track 0.00 -> 13.8 mm
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Other:
- board size 85.7 x 116 mm -> 85.7 x 113.5 mm
